File: PCB/key/plip/plip.kicad_pcb (KiCad board)
At the start: 2 copper layers, 1 part, among them IC1 PIC12F675-I_SN

Commit message: ???
Parts:
- added C1: TC212A476K006Y, test:TC212A476K006Y, F.Cu at (134.6, 68.6)
- added Q1: BSR16,215, test:BSR16,215, F.Cu at (134.0, 72.3)
- added R1: 0603WAF2203T5E, test:0603WAF2203T5E, F.Cu at (125.1, 74.8)
- IC1: footprint PIC12F675-I_SN:SOIC127P600X175-8N -> test:PIC12F675-I_SN
- moved IC1 34.1 mm to (127.4, 70.4)
Connections:
- IC1 pad 1: Net-(IC1-Pad1) -> unconnected-(IC1-Pad1)
- IC1 pad 2: Net-(IC1-Pad2) -> unconnected-(IC1-Pad2)
- IC1 pad 3: Net-(IC1-Pad3) -> unconnected-(IC1-Pad3)
- IC1 pad 4: Net-(IC1-Pad4) -> unconnected-(IC1-Pad4)
- IC1 pad 5: Net-(IC1-Pad5) -> unconnected-(IC1-Pad5)
- IC1 pad 6: Net-(IC1-Pad6) -> unconnected-(IC1-Pad6)
- IC1 pad 7: Net-(IC1-Pad7) -> unconnected-(IC1-Pad7)
- IC1 pad 8: Net-(IC1-Pad8) -> unconnected-(IC1-Pad8)
Other:
- net class Default removed

Commit message: add
Parts:
- removed C1: TC212A476K006Y, test:TC212A476K006Y
- removed R1: 0603WAF2203T5E, test:0603WAF2203T5E
- moved Q1 34.7 mm to (149.0, 41.0), turned to 90 degrees
- moved IC1 32.3 mm to (154.0, 52.0)
Connections:
- IC1 pad 1: unconnected-(IC1-Pad1) -> +5V
- IC1 pad 8: unconnected-(IC1-Pad8) -> GND
Other:
- board outline added: 28 x 21 mm
