File: PCB/key/plip/plip.kicad_sch (KiCad schematic)
At the start: 4 parts, among them IC1 PIC12F675-I_SN, Q1 BSR16,215

Commit message: add
Parts:
- removed C1: TC212A476K006Y, test:TC212A476K006Y, symbol test:TC212A476K006Y
- removed R1: 0603WAF2203T5E, test:0603WAF2203T5E, symbol test:0603WAF2203T5E
Connections:
- net +5V: now reaches IC1.1 (VDD)
- net GND: now reaches IC1.8 (VSS)
